Commit message: Gerçek robot saha betikleri, odom düzeltmesi, gerçekçi simülasyon
saha/: gerçek LIMO için haritalama, Nav2 (MPPI + AMCL), dikdörtgen tur ve robot
üzerinde rosbag kaydı (odom/IMU/lidar + Orbbec kamera). Kullanım: saha/README.md.
- robot/odom_duzelt.py: upstream sürücünün 0.1° yaw ölü bandını aşar (odom yönü
  IMU'dan); Nav2 sürüşünde yön hatası 23 m'de +73° -> +4.7° (docs/odom_analizi.md)
- dikdortgen.py: kenar boyunca düz, köşede yerinde dönüş; odom veya AMCL ile
- kayit_baslat/bitir.sh: robot diskine iki ayrı bag (sensor + kamera)
- nav_dur/harita_bitir: arka plan launch'lar SIGINT'i yok saydığı için INT->TERM

Simülasyon: gerçek ölçümlerle sensör gürültüsü (IMU, lidar), taban tepki modeli
(taban_modeli: gecikme + birinci derece + ivme sınırı), Ackermann teker teması,
myCobot eklemleri simde kilitli (kol çöküp lidarı kapatıyordu). docs/sensor_modeli.md.

Co-Authored-By: Claude Opus 5.5 <noreply@anthropic.com>

File: src/limo_car/gazebo/ackermann.xacro (robot description, xacro)
@@ -366,4 +366,10 @@
             </plugin>
         </gazebo>
+        <!-- Tekerlek teması (24.09): varsayılan ODE teması çok sert, araç dururken titriyordu
+             (IMU ivme σ z 0.25 m/s², gerçek 0.025). kp/kd sönümüyle gerçekle aynı (docs/sensor_modeli.md). -->
+        <gazebo reference="front_left_wheel_link"><mu1>1.0</mu1><mu2>1.0</mu2><kp>1000000.0</kp><kd>100.0</kd><minDepth>0.001</minDepth><maxVel>0.1</maxVel></gazebo>
+        <gazebo reference="front_right_wheel_link"><mu1>1.0</mu1><mu2>1.0</mu2><kp>1000000.0</kp><kd>100.0</kd><minDepth>0.001</minDepth><maxVel>0.1</maxVel></gazebo>
+        <gazebo reference="rear_left_wheel_link"><mu1>1.0</mu1><mu2>1.0</mu2><kp>1000000.0</kp><kd>100.0</kd><minDepth>0.001</minDepth><maxVel>0.1</maxVel></gazebo>
+        <gazebo reference="rear_right_wheel_link"><mu1>1.0</mu1><mu2>1.0</mu2><kp>1000000.0</kp><kd>100.0</kd><minDepth>0.001</minDepth><maxVel>0.1</maxVel></gazebo>
     </xacro:macro>
 </robot>

File: src/limo_car/gazebo/sensor.xacro (robot description, xacro)
@@ -40,19 +40,22 @@
         </link>
         <gazebo reference="${frame_prefix}_link">
+            <!-- Gerçek LIMO'dan ölçüldü (24.09, bag durağan aralıkları, docs/sensor_modeli.md): YDLIDAR T-mini
+     ~6 Hz, ~656 nokta/360°; arkada gövde/kol kapatıyor: etkin görüş -123°..+141°; menzil σ ≈ 4-6 mm (≤4 m),
+     12 mm (4-8 m) -> sabit 7 mm. Gazebo ışın kaybını (%5-10) modellemiyor. -->
             <sensor type="ray" name="laser_sensor">
                 <visualize>false</visualize>
-                <update_rate>8</update_rate>
+                <update_rate>6</update_rate>
                 <ray>
                     <scan>
                         <horizontal>
-                            <samples>720</samples>
+                            <samples>481</samples>
                             <resolution>1</resolution>
-                            <min_angle>-2.09439504</min_angle> <!-- Einheit in "rad", von Hersteller -->
-                            <max_angle>2.09439504</max_angle>
+                            <min_angle>-2.1468</min_angle> <!-- Einheit in "rad", von Hersteller -->
+                            <max_angle>2.4609</max_angle>
                         </horizontal>
                     </scan>
                     <range>
-                        <min>0.2</min>
-                        <max>8.0</max>
+                        <min>0.10</min>
+                        <max>12.0</max>
                         <resolution>0.01</resolution>
                     </range>
@@ -61,5 +64,5 @@
                         <type>gaussian</type>
                         <mean>0.0</mean>
-                        <stddev>0.01</stddev>
+                        <stddev>0.007</stddev>
                     </noise>
                 </ray>
@@ -187,17 +190,25 @@
             <gravity>true</gravity>
             <sensor name="imu_sensor" type="imu">
+                <!-- Gerçek LIMO IMU'su (24.09 ölçümü): ~92 Hz; jiroskop 0.1°/s nicemli, σ 0.00087 rad/s (y 0.0016);
+                     ivmeölçer σ 0.025 m/s². Eski blok ROS 1 etiketleri kullanıyordu (topicName, gaussianNoise) ->
+                     ROS 2 eklentisi yok sayıyordu, IMU gürültüsüzdü. -->
                 <always_on>true</always_on>
-                <update_rate>100</update_rate>
-                <visualize>true</visualize>
-                <topic>__default_topic__</topic>
-                <pose>0 0 0 0 0 0</pose>
+                <update_rate>90</update_rate>
+                <imu>
+                    <angular_velocity>
+                        <x><noise type="gaussian"><mean>0.0</mean><stddev>0.00087</stddev></noise></x>
+                        <y><noise type="gaussian"><mean>0.0</mean><stddev>0.0016</stddev></noise></y>
+                        <z><noise type="gaussian"><mean>0.0</mean><stddev>0.00087</stddev></noise></z>
+                    </angular_velocity>
+                    <linear_acceleration>
+                        <x><noise type="gaussian"><mean>0.0</mean><stddev>0.025</stddev></noise></x>
+                        <y><noise type="gaussian"><mean>0.0</mean><stddev>0.025</stddev></noise></y>
+                        <z><noise type="gaussian"><mean>0.0</mean><stddev>0.025</stddev></noise></z>
+                    </linear_acceleration>
+                </imu>
                 <plugin filename="libgazebo_ros_imu_sensor.so" name="imu_plugin">
-                    <topicName>/limo/imu</topicName>
-                    <bodyName>${frame_prefix}_link</bodyName>
-                    <updateRateHZ>100.0</updateRateHZ>
-                    <gaussianNoise>0.001</gaussianNoise>
-                    <xyzOffset>0 0 0</xyzOffset>
-                    <rpyOffset>0 0 0</rpyOffset>
-                    <frameName>${frame_prefix}_link</frameName>
+                    <ros><namespace>/</namespace><remapping>~/out:=imu</remapping></ros>
+                    <frame_name>${frame_prefix}_link</frame_name>
+                    <initial_orientation_as_reference>false</initial_orientation_as_reference>
                 </plugin>
             </sensor>

File: src/limo_description/urdf/limo_four_diff.xacro (robot description, xacro)
@@ -74,7 +74,9 @@
     <gazebo reference="imu_link">
     <gravity>true</gravity>
+    <!-- Gerçek LIMO IMU'su (24.09 ölçümü): ~92 Hz, jiroskop σ 0.00087 rad/s (0.1°/s nicemli; y 0.0016),
+         ivmeölçer σ 0.025 m/s², duruşta yön kayması ~0. Konu gerçekteki gibi /imu. -->
     <sensor name="twr_imu" type="imu">
       <always_on>true</always_on>
-      <update_rate>100</update_rate>
+      <update_rate>90</update_rate>
       <visualize>true</visualize>
       <imu>
@@ -83,5 +85,5 @@
             <noise type="gaussian">
               <mean>0.0</mean>
-              <stddev>2e-3</stddev>
+              <stddev>1e-4</stddev>
             </noise>
           </x>
@@ -89,5 +91,5 @@
             <noise type="gaussian">
               <mean>0.0</mean>
-              <stddev>2e-3</stddev>
+              <stddev>1e-4</stddev>
             </noise>
           </y>
@@ -95,5 +97,5 @@
             <noise type="gaussian">
               <mean>0.0</mean>
-              <stddev>2e-3</stddev>
+              <stddev>1e-4</stddev>
             </noise>
           </z>
@@ -103,5 +105,5 @@
             <noise type="gaussian">
               <mean>0.0</mean>
-              <stddev>2e-4</stddev>
+              <stddev>0.00087</stddev>
             </noise>
           </x>
@@ -109,5 +111,5 @@
             <noise type="gaussian">
               <mean>0.0</mean>
-              <stddev>2e-4</stddev>
+              <stddev>0.0016</stddev>
             </noise>
           </y>
@@ -115,5 +117,5 @@
             <noise type="gaussian">
               <mean>0.0</mean>
-              <stddev>2e-4</stddev>
+              <stddev>0.00087</stddev>
             </noise>
           </z>
@@ -123,5 +125,5 @@
             <noise type="gaussian">
               <mean>0.0</mean>
-              <stddev>1.7e-2</stddev>
+              <stddev>0.025</stddev>
             </noise>
           </x>
@@ -129,5 +131,5 @@
             <noise type="gaussian">
               <mean>0.0</mean>
-              <stddev>1.7e-2</stddev>
+              <stddev>0.025</stddev>
             </noise>
           </y>
@@ -135,5 +137,5 @@
             <noise type="gaussian">
               <mean>0.0</mean>
-              <stddev>1.7e-2</stddev>
+              <stddev>0.025</stddev>
             </noise>
           </z>
@@ -144,6 +146,6 @@
         <frame_name>imu_link</frame_name>
         <ros>
-          <namespace>/imu</namespace>
-          <remapping>~/out:=data</remapping>
+          <namespace>/</namespace>
+          <remapping>~/out:=imu</remapping>
         </ros>
       </plugin>
@@ -151,20 +153,23 @@
 </gazebo>
 <gazebo reference="laser_link">
+    <!-- Gerçek LIMO'dan ölçüldü (24.09, bag durağan aralıkları, docs/sensor_modeli.md): YDLIDAR T-mini
+     ~6 Hz, ~656 nokta/360°; arkada gövde/kol kapatıyor: etkin görüş -123°..+141°; menzil σ ≈ 4-6 mm (≤4 m),
+     12 mm (4-8 m) -> sabit 7 mm. Gazebo ışın kaybını (%5-10) modellemiyor. -->
     <sensor name="laser" type="ray">
       <always_on>true</always_on>
       <visualize>true</visualize>
-      <update_rate>10</update_rate>
+      <update_rate>6</update_rate>
       <ray>
         <scan>
           <horizontal>
-            <samples>120</samples>
+            <samples>481</samples>
             <resolution>1.000000</resolution>
-            <min_angle>-3.14159</min_angle>
-            <max_angle>3.14159</max_angle>
+            <min_angle>-2.1468</min_angle>
+            <max_angle>2.4609</max_angle>
           </horizontal>
         </scan>
         <range>
-          <min>0.3</min>
-          <max>15.0</max>
+          <min>0.10</min>
+          <max>12.0</max>
           <resolution>0.015</resolution>
         </range>
@@ -172,5 +177,5 @@
           <type>gaussian</type>
           <mean>0.0</mean>
-          <stddev>0.01</stddev>
+          <stddev>0.007</stddev>
         </noise>
       </ray>
@@ -232,4 +237,6 @@
              0.64 -> 0.31, salınım 3.7 -> 1.8 /m, tur 110 -> 87 s (bench/diffwobble). -->
         <plugin name="planar_move" filename="libgazebo_ros_planar_move.so">
+            <!-- Komut gerçek taban modelinden geçer (limo_kinematics/taban_modeli): /cmd_vel -> cmd_vel_taban -->
+            <ros><remapping>cmd_vel:=cmd_vel_taban</remapping></ros>
             <update_rate>50</update_rate>
             <publish_rate>50</publish_rate>

File: src/mycobot_description/urdf/mycobot/mycobot.urdf.xacro (robot description, xacro)
@@ -1,4 +1,9 @@
 <?xml version="1.0"?>
 <robot xmlns:xacro="http://www.ros.org/wiki/xacro" name="mycobot_280">
+  <!-- kol_kilit:=true -> eklemler fixed. Gazebo'da kolu tutan bir kontrolcü yok; revolute eklemler yalnızca
+       sürtünmeyle duruyor ve robot hareket ettikçe kol çöküp lidar düzlemine giriyordu (24 ileri/dönüş döngüsünde
+       uç z 0.56 -> 0.12 m; Nav2 önünde kalıcı sahte engel gördü). Gerçekte servolar kolu tutar. -->
+  <xacro:arg name="kol_kilit" default="false"/>
+  <xacro:property name="kol_eklem" value="${'fixed' if '$(arg kol_kilit)' == 'true' else 'revolute'}"/>
   <!-- Link 1 (Base of the arm) -->
   <link name="joint1">
@@ -22,5 +27,5 @@
   </link>
   <!-- Joint 1 to 2 (-168 to +168 deg) -->
-  <joint name="joint2_to_joint1" type="revolute">
+  <joint name="joint2_to_joint1" type="${kol_eklem}">
     <axis xyz="0 0 1"/>
     <limit effort="10.0" lower="-2.9322" upper="2.9322" velocity="1.5"/>
@@ -51,5 +56,5 @@
   </link>
   <!-- Joint 2 to 3 (-135 to +135 deg) -->
-  <joint name="joint3_to_joint2" type="revolute">
+  <joint name="joint3_to_joint2" type="${kol_eklem}">
     <axis xyz="0 0 1"/>
     <limit effort="10.0" lower="-2.3562" upper="2.3562" velocity="1.5"/>
@@ -80,5 +85,5 @@
   </link>
   <!-- Joint 3 to 4 (-150 to +150 deg) -->
-  <joint name="joint4_to_joint3" type="revolute">
+  <joint name="joint4_to_joint3" type="${kol_eklem}">
     <axis xyz="0 0 1"/>
     <limit effort="10.0" lower="-2.6180" upper="2.6180" velocity="1.5"/>
@@ -109,5 +114,5 @@
   </link>
   <!-- Joint 4 to 5 (-145 to +145 deg) -->
-  <joint name="joint5_to_joint4" type="revolute">
+  <joint name="joint5_to_joint4" type="${kol_eklem}">
     <axis xyz="0 0 1"/>
     <limit effort="10.0" lower="-2.5307" upper="2.5307" velocity="1.5"/>
@@ -138,5 +143,5 @@
   </link>
   <!-- Joint 5 to 6 (-165 to +165 deg) -->
-  <joint name="joint6_to_joint5" type="revolute">
+  <joint name="joint6_to_joint5" type="${kol_eklem}">
     <axis xyz="0 0 1"/>
     <limit effort="10.0" lower="-2.8798" upper="2.8798" velocity="1.5"/>
@@ -167,5 +172,5 @@
   </link>
   <!-- Joint 6 to 6_flange (-175 to +175 deg) -->
-  <joint name="joint6output_to_joint6" type="revolute">
+  <joint name="joint6output_to_joint6" type="${kol_eklem}">
     <axis xyz="0 0 1"/>
     <limit effort="10.0" lower="-3.0543" upper="3.0543" velocity="1.5"/>
