Commit message: Kamera dış kalibrasyonu: resmi AgileX değeri (base_link -> camera_link 0.084, 0, 0.03)
URDF'lerdeki kamera konumu (0.105, 0, 0.1) resmi değere çekildi; saha betikleri
base_link -> camera_link statik TF'ini yayınlıyor (Orbbec sürücüsü bu halkayı
vermiyor), config/kamera_kalibrasyon.yaml çerçeve zincirini ve kare pozu formülünü
belgeliyor.

Co-Authored-By: Claude Opus 5.5 <noreply@anthropic.com>

File: src/limo_car/gazebo/ackermann_with_sensor.xacro (robot description, xacro)
@@ -25,5 +25,6 @@
     <xacro:gazebo_depth_camera frame_prefix="camera" />
     <joint name="depth_camera_joint" type="fixed">
-        <origin xyz="0.105 0 0.1" rpy="0 0 0"/>
+        <!-- resmi AgileX değeri (bkz. limo_description/urdf/limo_four_diff.xacro) -->
+        <origin xyz="0.084 0 0.03" rpy="0 0 0"/>
         <parent link="base_link"/>
         <child link="camera_link"/>

File: src/limo_description/urdf/limo_ackerman.xacro (robot description, xacro)
@@ -55,6 +55,8 @@
         <origin xyz="0.105 0 0.08" rpy="0 0 -0.15"/>
     </xacro:limo_laser>
+    <!-- Resmi AgileX URDF (limo_description, limo_ros1): base_link -> derinlik kamerası (0.084, 0, 0.03), eğimsiz;
+         base_link yerden 0.15 m -> kamera ~0.18 m (09.10 sahada doğrulandı: yatay, lidar ile aynı yöne bakıyor). -->
     <xacro:limo_depth_camera parent_prefix="base_link" frame_prefix="camera">
-        <origin xyz="0.105 0 0.1" rpy="0 0 0"/>
+        <origin xyz="0.084 0 0.03" rpy="0 0 0"/>
     </xacro:limo_depth_camera>
     <xacro:limo_imu parent_prefix="base_link" frame_prefix="imu">

File: src/limo_description/urdf/limo_four_diff.xacro (robot description, xacro)
@@ -54,6 +54,8 @@
         <origin xyz="0.105 0 0.08" rpy="0 0 -0.15"/>
     </xacro:limo_laser>
+    <!-- Resmi AgileX URDF (limo_description, limo_ros1): base_link -> derinlik kamerası (0.084, 0, 0.03), eğimsiz;
+         base_link yerden 0.15 m -> kamera ~0.18 m (09.10 sahada doğrulandı: yatay, lidar ile aynı yöne bakıyor). -->
     <xacro:limo_depth_camera parent_prefix="base_link" frame_prefix="camera">
-        <origin xyz="0.105 0 0.1" rpy="0 0 0"/>
+        <origin xyz="0.084 0 0.03" rpy="0 0 0"/>
     </xacro:limo_depth_camera>
     <xacro:limo_imu parent_prefix="base_link" frame_prefix="imu">
